File: matrix.sch (KiCad schematic (older format))
At the start: 134 parts, among them SW1 SW_Push, SW10 SW_Push, SW11 SW_Push, SW12 SW_Push, SW13 SW_Push, SW14 SW_Push, SW15 SW_Push, SW16 SW_Push, SW17 SW_Push, SW18 SW_Push, SW19 SW_Push, SW2 SW_Push, SW20 SW_Push, SW21 SW_Push, SW22 SW_Push, SW23 SW_Push, SW24 SW_Push, SW25 SW_Push, SW26 SW_Push, SW27 SW_Push, SW28 SW_Push, SW29 SW_Push, SW3 SW_Push, SW30 SW_Push, SW31 SW_Push, SW32 SW_Push, SW33 SW_Push, SW34 SW_Push, SW35 SW_Push, SW36 SW_Push, SW37 SW_Push, SW38 SW_Push, SW39 SW_Push, SW4 SW_Push, SW40 SW_Push, SW41 SW_Push, SW42 SW_Push, SW43 SW_Push, SW44 SW_Push, SW45 SW_Push, SW46 SW_Push, SW47 SW_Push, SW48 SW_Push, SW49 SW_Push, SW5 SW_Push, SW50 SW_Push, SW51 SW_Push, SW52 SW_Push, SW53 SW_Push, SW54 SW_Push, SW55 SW_Push, SW56 SW_Push, SW57 SW_Push, SW58 SW_Push, SW59 SW_Push, SW6 SW_Push, SW60 SW_Push, SW61 SW_Push, SW62 SW_Push, SW63 SW_Push, SW64 SW_Push, SW65 SW_Push, SW66 SW_Push, SW67 SW_Push, SW7 SW_Push, SW8 SW_Push, SW9 SW_Push

Commit message: Assign PCB footprints to schematic symbols
Parts:
- D1, D10, D11, D12, D13, D14, D15, D16, D17, D18, D19, D2, D20, D21, D22, D23, D24, D25, D26, D27, D28, D29, D3, D30, D31, D32, D33, D34, D35, D36, D37, D38, D39, D4, D40, D41, D42, D43, D44, D45, D46, D47, D48, D49, D5, D50, D51, D52, D53, D54, D55, D56, D57, D58, D59, D6, D60, D61, D62, D63, D64, D65, D66, D67, D7, D8, D9: footprint (none) -> Diodes_SMD:D_SOD-123
- SW1, SW10, SW11, SW12, SW13, SW15, SW16, SW17, SW18, SW19, SW20, SW21, SW22, SW24, SW25, SW26, SW27, SW28, SW29, SW30, SW31, SW32, SW33, SW34, SW35, SW36, SW38, SW39, SW40, SW41, SW42, SW43, SW44, SW45, SW47, SW48, SW49, SW50, SW51, SW52, SW53, SW55, SW56, SW58, SW59, SW6, SW61, SW62, SW63, SW64, SW65, SW66, SW67, SW7, SW8, SW9: footprint (none) -> Fate_Parts:SW_Cherry_MX_1.00u_PCB
- SW14, SW2, SW46, SW5, SW60: footprint (none) -> Fate_Parts:SW_Cherry_MX_1.50u_PCB
- SW23: footprint (none) -> Fate_Parts:SW_Cherry_MX_2.00u_PCB_ReversedStabilizers
- SW3, SW54: footprint (none) -> Fate_Parts:SW_Cherry_MX_1.75u_PCB
- SW37: footprint (none) -> Fate_Parts:SW_Cherry_MX_2.75u_PCB_ReversedStabilizers
- SW4: footprint (none) -> Fate_Parts:SW_Cherry_MX_2.25u_PCB
- SW57: footprint (none) -> Fate_Parts:SW_Cherry_MX_2.25u_PCB_ReversedStabilizers
