File: arisu.kicad_pcb (KiCad board)
At the start: 2 copper layers, 339.1 x 118.7 mm, 166 parts, among them J1 USB_B_Micro, SW1 SW_Push, SW10 SW_Push, SW11 SW_Push, SW12 SW_Push, SW13 SW_Push, SW14 SW_Push, SW15 SW_Push, SW16 SW_Push, SW17 SW_Push, SW18 SW_Push, SW19 SW_Push, SW2 SW_Push, SW20 SW_Push, SW21 SW_Push, SW22 SW_Push, SW23 SW_Push, SW24 SW_Push, SW25 SW_Push, SW26 SW_Push, SW27 SW_Push, SW28 SW_Push, SW29 SW_Push, SW3 SW_Push, SW30 SW_Push, SW31 SW_Push, SW32 SW_Push, SW33 SW_Push, SW34 SW_Push, SW35 SW_Push, SW36 SW_Push, SW37 SW_Push, SW38 SW_Push, SW39 SW_Push, SW4 SW_Push, SW40 SW_Push, SW41 SW_Push, SW42 SW_Push, SW43 SW_Push, SW44 SW_Push, SW45 SW_Push, SW46 SW_Push, SW47 SW_Push, SW48 SW_Push, SW49 SW_Push, SW5 SW_Push, SW50 SW_Push, SW51 SW_Push, SW52 SW_Push, SW53 SW_Push, SW54 SW_Push, SW55 SW_Push, SW56 SW_Push, SW57 SW_Push, SW58 SW_Push, SW59 SW_Push, SW6 SW_Push, SW60 SW_Push, SW61 SW_Push, SW62 SW_Push, SW63 SW_Push, SW64 SW_Push, SW65 SW_Push, SW66 SW_Push, SW67 SW_Push, SW7 SW_Push, SW8 SW_Push, SW9 SW_Push, U1 USBLC6-2SC6, U2 ATmega32U4-AU, Y1 Crystal_GND24

Commit message: Add Arisu Logo
Parts:
- added G***: LOGO, arisu:arisu-logo, B.Cu at (287.0, 114.9)
- added G***: LOGO, arisu:arisu-logo, F.Cu at (287.0, 117.3)
Other:
- board text added: "Fate Design Rev 1.0"

Commit message: Add mounting holes in PCBNew
Parts:
- added H1: MountingHole, Mounting_Holes:MountingHole_2.2mm_M2_Pad, F.Cu at (56.9, 48.2)
- added H2: MountingHole, Mounting_Holes:MountingHole_2.2mm_M2_Pad, F.Cu at (51.2, 114.9)
- added H3: MountingHole, Mounting_Holes:MountingHole_2.2mm_M2_Pad, F.Cu at (121.8, 27.9)
- added H4: MountingHole, Mounting_Holes:MountingHole_2.2mm_M2_Pad, F.Cu at (110.0, 120.6)
- added H5: MountingHole, Mounting_Holes:MountingHole_2.2mm_M2_Pad, F.Cu at (229.2, 27.9)
- added H6: MountingHole, Mounting_Holes:MountingHole_2.2mm_M2_Pad, F.Cu at (241.1, 120.6)
- added H7: MountingHole, Mounting_Holes:MountingHole_2.2mm_M2_Pad, F.Cu at (341.2, 43.5)
- added H8: MountingHole, Mounting_Holes:MountingHole_2.2mm_M2_Pad, F.Cu at (345.4, 110.2)
Routing:
- net /row1: track 383.4 -> 384.1 mm
Changed lines of the file:
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@@
     (thickness 1.6)
     (drawings 1381)
-    (tracks 880)
+    (tracks 884)
     (zones 0)
-    (modules 168)
+    (modules 176)
     (nets 108)
   )
@@
     (add_net VCC)
   )
+  (module Mounting_Holes:MountingHole_2.2mm_M2_Pad (layer F.Cu)
+    (at 241.060266 120.60872)
+    (descr "Mounting Hole 2.2mm, M2")
+    (tags "mounting hole 2.2mm m2")
+    (attr virtual)
+    (fp_text reference H6 (at 0 -3.2) (layer F.Fab)
+      (effects (font (size 1 1) (thickness 0.15)))
+    )
+    (fp_text value MountingHole (at 0 3.2) (layer F.Fab)
+      (effects (font (size 1 1) (thickness 0.15)))
+    )
+    (fp_text user %R (at 0.3 0) (layer F.Fab)
+      (effects (font (size 1 1) (thickness 0.15)))
+    )
+    (fp_circle (center 0 0) (end 2.2 0) (layer Cmts.User) (width 0.15))
+    (fp_circle (center 0 0) (end 2.45 0) (layer F.CrtYd) (width 0.05))
+    (pad 1 thru_hole circle (at 0 0) (size 4.4 4.4) (drill 2.2) (layers *.Cu *.Mask))
+  )
+  (module Mounting_Holes:MountingHole_2.2mm_M2_Pad (layer F.Cu)
+    (at 345.449949 110.157503)
+    (descr "Mounting Hole 2.2mm, M2")
+    (tags "mounting hole 2.2mm m2")
+    (attr virtual)
+    (fp_text reference H8 (at 0 -3.2) (layer F.Fab)
+      (effects (font (size 1 1) (thickness 0.15)))
+    )
+    (fp_text value MountingHole (at 0 3.2) (layer F.Fab)
+      (effects (font (size 1 1) (thickness 0.15)))
+    )
+    (fp_text user %R (at 0.3 0) (layer F.Fab)
+      (effects (font (size 1 1) (thickness 0.15)))
+    )
+    (fp_circle (center 0 0) (end 2.2 0) (layer Cmts.User) (width 0.15))
+    (fp_circle (center 0 0) (end 2.45 0) (layer F.CrtYd) (width 0.05))
+    (pad 1 thru_hole circle (at 0 0) (size 4.4 4.4) (drill 2.2) (layers *.Cu *.Mask))
+  )
   (module Capacitors_SMD:C_0805_HandSoldering (layer B.Cu)
     (at 185.166 40.894 270)
@@
       (xy 2.4511 -4.165596) (xy 3.048 -4.1656) (xy 3.046873 -2.9591)) (layer F.SilkS) (width 0.01))
   )
+  (module Mounting_Holes:MountingHole_2.2mm_M2_Pad (layer F.Cu)
+    (at 56.865 48.245)
+    (descr "Mounting Hole 2.2mm, M2")
+    (tags "mounting hole 2.2mm m2")
+    (attr virtual)
+    (fp_text reference H1 (at 0 -3.2) (layer F.SilkS)
+      (effects (font (size 1 1) (thickness 0.15)))
+    )
+    (fp_text value MountingHole (at 0 3.2) (layer F.Fab)
+      (effects (font (size 1 1) (thickness 0.15)))
+    )
+    (fp_circle (center 0 0) (end 2.45 0) (layer F.CrtYd) (width 0.05))
+    (fp_circle (center 0 0) (end 2.2 0) (layer Cmts.User) (width 0.15))
+    (fp_text user %R (at 0.3 0) (layer F.Fab)
+      (effects (font (size 1 1) (thickness 0.15)))
+    )
+    (pad 1 thru_hole circle (at 0 0) (size 4.4 4.4) (drill 2.2) (layers *.Cu *.Mask))
+  )
+  (module Mounting_Holes:MountingHole_2.2mm_M2_Pad (layer F.Cu)
+    (at 51.1975 114.92)
+    (descr "Mounting Hole 2.2mm, M2")
+    (tags "mounting hole 2.2mm m2")
+    (attr virtual)
+    (fp_text reference H2 (at 0 -3.2) (layer F.Fab)
+      (effects (font (size 1 1) (thickness 0.15)))
+    )
+    (fp_text value MountingHole (at 0 3.2) (layer F.Fab)
+      (effects (font (size 1 1) (thickness 0.15)))
+    )
+    (fp_text user %R (at 0.3 0) (layer F.Fab)
+      (effects (font (size 1 1) (thickness 0.15)))
+    )
+    (fp_circle (center 0 0) (end 2.2 0) (layer Cmts.User) (width 0.15))
+    (fp_circle (center 0 0) (end 2.45 0) (layer F.CrtYd) (width 0.05))
+    (pad 1 thru_hole circle (at 0 0) (size 4.4 4.4) (drill 2.2) (layers *.Cu *.Mask))
+  )
+  (module Mounting_Holes:MountingHole_2.2mm_M2_Pad (layer F.Cu)
+    (at 121.82722 27.932509)
+    (descr "Mounting Hole 2.2mm, M2")
+    (tags "mounting hole 2.2mm m2")
+    (attr virtual)
+    (fp_text reference H3 (at 0 -3.2) (layer F.Fab)
+      (effects (font (size 1 1) (thickness 0.15)))
+    )
+    (fp_text value MountingHole (at 0 3.2) (layer F.Fab)
+      (effects (font (size 1 1) (thickness 0.15)))
+    )
+    (fp_circle (center 0 0) (end 2.45 0) (layer F.CrtYd) (width 0.05))
+    (fp_circle (center 0 0) (end 2.2 0) (layer Cmts.User) (width 0.15))
+    (fp_text user %R (at 0.3 0) (layer F.Fab)
+      (effects (font (size 1 1) (thickness 0.15)))
+    )
+    (pad 1 thru_hole circle (at 0 0) (size 4.4 4.4) (drill 2.2) (layers *.Cu *.Mask))
+  )
+  (module Mounting_Holes:MountingHole_2.2mm_M2_Pad (layer F.Cu)
+    (at 109.959436 120.609368)
+    (descr "Mounting Hole 2.2mm, M2")
+    (tags "mounting hole 2.2mm m2")
+    (attr virtual)
+    (fp_text reference H4 (at 0 -3.2) (layer F.Fab)
+      (effects (font (size 1 1) (thickness 0.15)))
+    )
+    (fp_text value MountingHole (at 0 3.2) (layer F.Fab)
+      (effects (font (size 1 1) (thickness 0.15)))
+    )
+    (fp_text user %R (at 0.3 0) (layer F.Fab)
+      (effects (font (size 1 1) (thickness 0.15)))
+    )
+    (fp_circle (center 0 0) (end 2.2 0) (layer Cmts.User) (width 0.15))
+    (fp_circle (center 0 0) (end 2.45 0) (layer F.CrtYd) (width 0.05))
+    (pad 1 thru_hole circle (at 0 0) (size 4.4 4.4) (drill 2.2) (layers *.Cu *.Mask))
+  )
+  (module Mounting_Holes:MountingHole_2.2mm_M2_Pad (layer F.Cu)
+    (at 229.192785 27.932509)
+    (descr "Mounting Hole 2.2mm, M2")
+    (tags "mounting hole 2.2mm m2")
+    (attr virtual)
+    (fp_text reference H5 (at 0 -3.2) (layer F.Fab)
+      (effects (font (size 1 1) (thickness 0.15)))
+    )
+    (fp_text value MountingHole (at 0 3.2) (layer F.Fab)
+      (effects (font (size 1 1) (thickness 0.15)))
+    )
+    (fp_circle (center 0 0) (end 2.45 0) (layer F.CrtYd) (width 0.05))
+    (fp_circle (center 0 0) (end 2.2 0) (layer Cmts.User) (width 0.15))
+    (fp_text user %R (at 0.3 0) (layer F.Fab)
+      (effects (font (size 1 1) (thickness 0.15)))
+    )
+    (pad 1 thru_hole circle (at 0 0) (size 4.4 4.4) (drill 2.2) (layers *.Cu *.Mask))
+  )
+  (module Mounting_Holes:MountingHole_2.2mm_M2_Pad (layer F.Cu)
+    (at 341.18 43.482516)
+    (descr "Mounting Hole 2.2mm, M2")
+    (tags "mounting hole 2.2mm m2")
+    (attr virtual)
+    (fp_text reference H7 (at 0 -3.2) (layer F.Fab)
+      (effects (font (size 1 1) (thickness 0.15)))
+    )
+    (fp_text value MountingHole (at 0 3.2) (layer F.Fab)
+      (effects (font (size 1 1) (thickness 0.15)))
+    )
+    (fp_circle (center 0 0) (end 2.45 0) (layer F.CrtYd) (width 0.05))
+    (fp_circle (center 0 0) (end 2.2 0) (layer Cmts.User) (width 0.15))
+    (fp_text user %R (at 0.3 0) (layer F.Fab)
+      (effects (font (size 1 1) (thickness 0.15)))
+    )
+    (pad 1 thru_hole circle (at 0 0) (size 4.4 4.4) (drill 2.2) (layers *.Cu *.Mask))
+  )
   (gr_text "Fate Design Rev 1.0" (at 287.02 120.65) (layer B.SilkS)
     (effects (font (size 1.5 1.5) (thickness 0.3)) (justify mirror))
@@
   (segment (start 186.167195 75.952753) (end 182.206477 79.913471) (width 0.25) (layer B.Cu) (net 8))
   (segment (start 200.840188 75.952753) (end 186.167195 75.952753) (width 0.25) (layer B.Cu) (net 8))
-  (segment (start 318.905 63.195) (end 327.305 63.195) (width 0.25) (layer B.Cu) (net 8))
-  (segment (start 343.307542 47.192458) (end 343.307542 39.382509) (width 0.25) (layer B.Cu) (net 8))
-  (segment (start 327.305 63.195) (end 343.307542 47.192458) (width 0.25) (layer B.Cu) (net 8))
   (segment (start 257.616924 63.195) (end 256.741324 64.0706) (width 0.25) (layer B.Cu) (net 8))
   (segment (start 318.905 63.195) (end 257.616924 63.195) (width 0.25) (layer B.Cu) (net 8))
@@
   (segment (start 181.781001 44.024999) (end 194.098001 44.024999) (width 0.25) (layer F.Cu) (net 8))
   (segment (start 179.705 46.101) (end 181.781001 44.024999) (width 0.25) (layer F.Cu) (net 8))
+  (segment (start 326.949 63.195) (end 318.905 63.195) (width 0.25) (layer B.Cu) (net 8))
+  (segment (start 344.424 45.72) (end 326.949 63.195) (width 0.25) (layer B.Cu) (net 8))
+  (segment (start 344.424 41.198967) (end 344.424 45.72) (width 0.25) (layer B.Cu) (net 8))
+  (segment (start 343.307542 39.382509) (end 343.307542 40.082509) (width 0.25) (layer B.Cu) (net 8))
+  (segment (start 343.307542 40.082509) (end 344.424 41.198967) (width 0.25) (layer B.Cu) (net 8))
   (segment (start 44.715 55.815) (end 44.13 55.23) (width 0.375) (layer B.Cu) (net 9))
   (segment (start 44.715 59.895) (end 44.715 55.815) (width 0.375) (layer B.Cu) (net 9))
@@
   (segment (start 92.476829 120.345) (end 94.724247 122.592418) (width 0.375) (layer B.Cu) (net 15))
   (segment (start 36.485 120.345) (end 92.476829 120.345) (width 0.375) (layer B.Cu) (net 15))
-  (segment (start 120.401964 122.592418) (end 127.333239 129.523693) (width 0.375) (layer B.Cu) (net 15))
-  (segment (start 94.724247 122.592418) (end 120.401964 122.592418) (width 0.375) (layer B.Cu) (net 15))
   (segment (start 154.707226 134.888153) (end 155.283812 135.464739) (width 0.375) (layer B.Cu) (net 15))
   (segment (start 149.919352 130.100279) (end 154.707226 134.888153) (width 0.375) (layer B.Cu) (net 15))
@@
   (segment (start 223.462031 91.831236) (end 214.338774 82.707979) (width 0.25) (layer F.Cu) (net 15))
   (segment (start 214.338774 82.707979) (end 214.338774 76.525142) (width 0.25) (layer F.Cu) (net 15))
+  (segment (start 95.437651 122.592418) (end 98.575233 125.73) (width 0.25) (layer B.Cu) (net 15))
+  (segment (start 94.724247 122.592418) (end 95.437651 122.592418) (width 0.25) (layer B.Cu) (net 15))
+  (segment (start 123.539546 125.73) (end 127.333239 129.523693) (width 0.25) (layer B.Cu) (net 15))
+  (segment (start 98.575233 125.73) (end 123.539546 125.73) (width 0.25) (layer B.Cu) (net 15))
   (segment (start 63.165 36.765) (end 62.58 36.18) (width 0.375) (layer B.Cu) (net 16))
   (segment (start 63.165 40.845) (end 63.165 36.765) (width 0.375) (layer B.Cu) (net 16))
