File: arisu.kicad_pcb (KiCad board)
At the start: 2 copper layers, 339.1 x 118.7 mm, 176 parts, among them J1 USB_B_Micro, SW1 SW_Push, SW10 SW_Push, SW11 SW_Push, SW12 SW_Push, SW13 SW_Push, SW14 SW_Push, SW15 SW_Push, SW16 SW_Push, SW17 SW_Push, SW18 SW_Push, SW19 SW_Push, SW2 SW_Push, SW20 SW_Push, SW21 SW_Push, SW22 SW_Push, SW23 SW_Push, SW24 SW_Push, SW25 SW_Push, SW26 SW_Push, SW27 SW_Push, SW28 SW_Push, SW29 SW_Push, SW3 SW_Push, SW30 SW_Push, SW31 SW_Push, SW32 SW_Push, SW33 SW_Push, SW34 SW_Push, SW35 SW_Push, SW36 SW_Push, SW37 SW_Push, SW38 SW_Push, SW39 SW_Push, SW4 SW_Push, SW40 SW_Push, SW41 SW_Push, SW42 SW_Push, SW43 SW_Push, SW44 SW_Push, SW45 SW_Push, SW46 SW_Push, SW47 SW_Push, SW48 SW_Push, SW49 SW_Push, SW5 SW_Push, SW50 SW_Push, SW51 SW_Push, SW52 SW_Push, SW53 SW_Push, SW54 SW_Push, SW55 SW_Push, SW56 SW_Push, SW57 SW_Push, SW58 SW_Push, SW59 SW_Push, SW6 SW_Push, SW60 SW_Push, SW61 SW_Push, SW62 SW_Push, SW63 SW_Push, SW64 SW_Push, SW65 SW_Push, SW66 SW_Push, SW67 SW_Push, SW7 SW_Push, SW8 SW_Push, SW9 SW_Push, U1 USBLC6-2SC6, U2 ATmega32U4-AU, Y1 Crystal_GND24

Commit message: Increase D+ and D- differential pair track width
Routing:
- net /col6: track 97.9 -> 96.8 mm

Commit message: Add ground fill zone on B.Cu
Routing:
- net /col11: track 224.6 -> 230.6 mm
Other:
- board text added: "Fate Design Rev 1.1"
- board text removed: "Fate Design Rev 1.0"
Changed lines of the file:
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@@
     (thickness 1.6)
     (drawings 1381)
-    (tracks 843)
+    (tracks 855)
     (zones 0)
     (modules 176)
@@
   )
   (page User 389.992 200)
+  (title_block
+    (rev 1.1)
+  )
   (layers
     (0 F.Cu signal)
@@
     (pad 1 thru_hole circle (at 0 0) (size 4.4 4.4) (drill 2.2) (layers *.Cu *.Mask))
   )
-  (gr_text "Fate Design Rev 1.0" (at 287.02 120.65) (layer B.SilkS)
+  (gr_text "Fate Design Rev 1.1" (at 287.02 120.65) (layer B.SilkS)
     (effects (font (size 1.5 1.5) (thickness 0.3)) (justify mirror))
   )
@@
   (segment (start 271.79 71.74) (end 271.79 81.264979) (width 0.25) (layer F.Cu) (net 101) (status 10))
   (segment (start 280.21502 89.689999) (end 281.315019 90.789998) (width 0.25) (layer B.Cu) (net 101) (status 20))
-  (segment (start 229.499219 89.689999) (end 280.21502 89.689999) (width 0.25) (layer B.Cu) (net 101))
-  (segment (start 220.742272 98.446946) (end 229.499219 89.689999) (width 0.25) (layer B.Cu) (net 101))
-  (segment (start 190.197645 98.446946) (end 220.742272 98.446946) (width 0.25) (layer B.Cu) (net 101))
-  (segment (start 174.714 82.963301) (end 190.197645 98.446946) (width 0.25) (layer B.Cu) (net 101))
   (segment (start 174.714 47.864) (end 174.714 82.963301) (width 0.25) (layer B.Cu) (net 101) (status 10))
+  (segment (start 174.714 82.963301) (end 190.197645 98.446946) (width 0.25) (layer B.Cu) (net 101))
+  (segment (start 190.197645 98.446946) (end 211.553054 98.446946) (width 0.25) (layer B.Cu) (net 101))
+  (segment (start 211.553054 98.446946) (end 216 94) (width 0.25) (layer B.Cu) (net 101))
+  (segment (start 236.379998 94) (end 240.689999 89.689999) (width 0.25) (layer B.Cu) (net 101))
+  (segment (start 216 94) (end 236.379998 94) (width 0.25) (layer B.Cu) (net 101))
+  (segment (start 240.689999 89.689999) (end 280.21502 89.689999) (width 0.25) (layer B.Cu) (net 101))
   (segment (start 268.11 39) (end 281.8 52.69) (width 0.25) (layer F.Cu) (net 102) (status 20))
   (segment (start 268.11 32.139615) (end 268.11 39) (width 0.25) (layer F.Cu) (net 102) (status 10))
@@
   (segment (start 307.508769 88.408769) (end 290.84 71.74) (width 0.25) (layer F.Cu) (net 102) (status 20))
   (segment (start 307.508769 90.789998) (end 307.508769 88.408769) (width 0.25) (layer F.Cu) (net 102) (status 10))
-  (segment (start 289.414999 70.314999) (end 290.84 71.74) (width 0.25) (layer B.Cu) (net 102) (status 20))
-  (segment (start 222.611545 70.314999) (end 289.414999 70.314999) (width 0.25) (layer B.Cu) (net 102))
-  (segment (start 212.12315 80.803394) (end 222.611545 70.314999) (width 0.25) (layer B.Cu) (net 102))
-  (segment (start 181.578524 80.803394) (end 212.12315 80.803394) (width 0.25) (layer B.Cu) (net 102))
-  (segment (start 175.514 74.73887) (end 181.578524 80.803394) (width 0.25) (layer B.Cu) (net 102))
-  (segment (start 175.514 47.864) (end 175.514 74.73887) (width 0.25) (layer B.Cu) (net 102) (status 10))
+  (segment (start 289.1 70) (end 290.84 71.74) (width 0.25) (layer B.Cu) (net 102) (status 20))
+  (segment (start 250 70) (end 289.1 70) (width 0.25) (layer B.Cu) (net 102))
+  (segment (start 231 74) (end 246 74) (width 0.25) (layer B.Cu) (net 102))
+  (segment (start 227 78) (end 231 74) (width 0.25) (layer B.Cu) (net 102))
+  (segment (start 246 74) (end 250 70) (width 0.25) (layer B.Cu) (net 102))
+  (segment (start 175.514 78.514) (end 182 85) (width 0.25) (layer B.Cu) (net 102))
+  (segment (start 175.514 47.864) (end 175.514 78.514) (width 0.25) (layer B.Cu) (net 102) (status 10))
+  (segment (start 182 85) (end 190 85) (width 0.25) (layer B.Cu) (net 102))
+  (segment (start 213 78) (end 227 78) (width 0.25) (layer B.Cu) (net 102))
+  (segment (start 190 85) (end 193 82) (width 0.25) (layer B.Cu) (net 102))
+  (segment (start 193 82) (end 209 82) (width 0.25) (layer B.Cu) (net 102))
+  (segment (start 209 82) (end 213 78) (width 0.25) (layer B.Cu) (net 102))
   (segment (start 287.16 39) (end 300.85 52.69) (width 0.25) (layer F.Cu) (net 103) (status 20))
   (segment (start 287.16 33.64) (end 287.16 39) (width 0.25) (layer F.Cu) (net 103) (status 10))
@@
   (segment (start 183.415156 70.31395) (end 193.313034 70.31395) (width 0.25) (layer B.Cu) (net 103))
   (segment (start 259.732844 50.95001) (end 299.11001 50.95001) (width 0.25) (layer B.Cu) (net 103))
-  (segment (start 193.313034 70.31395) (end 210.909114 52.71787) (width 0.25) (layer B.Cu) (net 103))
-  (segment (start 210.909114 52.71787) (end 257.964984 52.71787) (width 0.25) (layer B.Cu) (net 103))
   (segment (start 257.964984 52.71787) (end 259.732844 50.95001) (width 0.25) (layer B.Cu) (net 103))
+  (segment (start 257.964984 52.71787) (end 235.28213 52.71787) (width 0.25) (layer B.Cu) (net 103))
+  (segment (start 229.186508 58.813492) (end 204.813492 58.813492) (width 0.25) (layer B.Cu) (net 103))
+  (segment (start 235.28213 52.71787) (end 229.186508 58.813492) (width 0.25) (layer B.Cu) (net 103))
+  (segment (start 193.313034 70.31395) (end 204.813492 58.813492) (width 0.25) (layer B.Cu) (net 103))
   (segment (start 324.67 52.1) (end 324.67 52.69) (width 0.25) (layer F.Cu) (net 104) (status 30))
   (segment (start 306.21 33.64) (end 324.67 52.1) (width 0.25) (layer F.Cu) (net 104) (status 30))
@@
   (segment (start 324.67 52.69) (end 338.464949 66.484949) (width 0.25) (layer F.Cu) (net 104) (status 10))
   (segment (start 338.464949 95.552503) (end 338.464949 114.602503) (width 0.25) (layer F.Cu) (net 104) (status 30))
-  (segment (start 177.114 63.376384) (end 183.601556 69.86394) (width 0.25) (layer B.Cu) (net 104))
+  (segment (start 322.48 50.5) (end 324.67 52.69) (width 0.25) (layer B.Cu) (net 104) (status 20))
+  (segment (start 257.778584 52.26786) (end 259.546444 50.5) (width 0.25) (layer B.Cu) (net 104))
+  (segment (start 235.095729 52.267861) (end 257.778584 52.26786) (width 0.25) (layer B.Cu) (net 104))
   (segment (start 177.114 47.864) (end 177.114 63.376384) (width 0.25) (layer B.Cu) (net 104) (status 10))
-  (segment (start 210.722714 52.26786) (end 193.126634 69.86394) (width 0.25) (layer B.Cu) (net 104))
-  (segment (start 324.67 52.69) (end 322.48 50.5) (width 0.25) (layer B.Cu) (net 104) (status 10))
-  (segment (start 322.48 50.5) (end 259.546444 50.5) (width 0.25) (layer B.Cu) (net 104))
-  (segment (start 259.546444 50.5) (end 257.778584 52.26786) (width 0.25) (layer B.Cu) (net 104))
-  (segment (start 257.778584 52.26786) (end 210.722714 52.26786) (width 0.25) (layer B.Cu) (net 104))
+  (segment (start 177.114 63.376384) (end 183.601556 69.86394) (width 0.25) (layer B.Cu) (net 104))
   (segment (start 183.601556 69.86394) (end 193.126634 69.86394) (width 0.25) (layer B.Cu) (net 104))
+  (segment (start 193.126634 69.86394) (end 204.627091 58.363483) (width 0.25) (layer B.Cu) (net 104))
+  (segment (start 204.627091 58.363483) (end 229.000108 58.363482) (width 0.25) (layer B.Cu) (net 104))
+  (segment (start 259.546444 50.5) (end 322.48 50.5) (width 0.25) (layer B.Cu) (net 104))
+  (segment (start 229.000108 58.363482) (end 235.095729 52.267861) (width 0.25) (layer B.Cu) (net 104))
   (zone (net 1) (net_name GND) (layer B.Cu) (hatch edge 0.508)
     (connect_pads (clearance 0.508))
@@
     (connect_pads (clearance 0.508))
     (min_thickness 0.254)
+    (fill yes (arc_segments 32) (thermal_gap 0.508) (thermal_bridge_width 0.508))
+    (polygon
+      (pts
+        (xy 22.86 22.86) (xy 368.3 22.86) (xy 368.3 144.78) (xy 22.86 144.78)
+      )
+    )
+  )
+  (zone (net 1) (net_name GND) (layer B.Cu) (hatch edge 0.508)
+    (connect_pads (clearance 0.508))
+    (min_thickness 0.254)
